Commit message: working admittance in simulation

File: ur_description/urdf/ur_macro.xacro (robot description, xacro)
@@ -314,4 +314,10 @@
       <dynamics damping="0" friction="0"/>
     </joint>
+      <link name="${prefix}ft_frame"/>
+        <joint name="${prefix}wrist_3_link-ft_frame" type="fixed">
+          <parent link="${prefix}wrist_3_link"/>
+          <child link="${prefix}ft_frame"/>
+          <origin xyz="0 0 0" rpy="${pi} 0 0"/>
+        </joint>
     <!-- ROS-Industrial 'base' frame - base_link to UR 'Base' Coordinates transform -->
     <link name="${prefix}base"/>
